File: HighSideSwitchModule.kicad_sch (KiCad schematic)
At the start: 8 parts, among them J1 M3, J2 M3, J3 M3, J4 M3, J5 Input

Commit message: Fixed FETs on input.
Changed lines of the file:
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@@
   (junction (at 103.632 72.39) (diameter 0) (color 0 0 0 0)
-  )
-  (wire (pts (xy 114.554 75.438) (xy 114.554 42.926))
-    (stroke (width 0) (type default))
   )
   (wire (pts (xy 236.855 144.145) (xy 236.855 148.59))
@@
     (stroke (width 0) (type default))
   )
+  (wire (pts (xy 114.554 42.926) (xy 114.554 75.438))
+    (stroke (width 0) (type default))
+  )
